Commit message: final update

File: description/example_include.xacro (robot description, xacro)
@@ -1,5 +1,5 @@
 <?xml version="1.0"?>
-<robot xmlns:xacro="http://www.ros.org/wiki/xacro">
-     <!-- This file is not a robot in and of itself, it just contains some useful tags that could be included in any robot -->
+<robot xmlns:xacro="http://www.ros.org/wiki/xacro" >
+    <!-- This file is not a robot in and of itself, it just contains some useful tags that could be included in any robot -->
     <!-- Specify some colours -->
     <material name="white">
@@ -17,8 +17,8 @@
         <inertial>
             <xacro:insert_block name="origin"/>
-            <mass value="${mass}"/>
+            <mass value="${mass}" />
             <inertia ixx="${(2/5) * mass * (radius*radius)}" ixy="0.0" ixz="0.0"
                     iyy="${(2/5) * mass * (radius*radius)}" iyz="0.0"
-                    izz="${(2/5) * mass * (radius*radius)}"/>
+                    izz="${(2/5) * mass * (radius*radius)}" />
         </inertial>
     </xacro:macro>
@@ -26,8 +26,8 @@
         <inertial>
             <xacro:insert_block name="origin"/>
-            <mass value="${mass}"/>
+            <mass value="${mass}" />
             <inertia ixx="${(1/12) * mass * (y*y+z*z)}" ixy="0.0" ixz="0.0"
                     iyy="${(1/12) * mass * (x*x+z*z)}" iyz="0.0"
-                    izz="${(1/12) * mass * (x*x+y*y)}"/>
+                    izz="${(1/12) * mass * (x*x+y*y)}" />
         </inertial>
     </xacro:macro>
@@ -35,8 +35,8 @@
         <inertial>
             <xacro:insert_block name="origin"/>
-            <mass value="${mass}"/>
+            <mass value="${mass}" />
             <inertia ixx="${(1/12) * mass * (3*radius*radius + length*length)}" ixy="0.0" ixz="0.0"
                     iyy="${(1/12) * mass * (3*radius*radius + length*length)}" iyz="0.0"
-                    izz="${(1/2) * mass * (radius*radius)}"/>
+                    izz="${(1/2) * mass * (radius*radius)}" />
         </inertial>
     </xacro:macro>

File: description/example_robot.urdf.xacro (robot description, xacro)
@@ -1,4 +1,4 @@
 <?xml version="1.0"?>
-<robot xmlns:xacro="http://www.ros.org/wiki/xacro" name="robot">
+<robot xmlns:xacro="http://www.ros.org/wiki/xacro"  name="robot">
     <!-- This is an example of a URDF. -->
     <!-- As we move through the file, new things to note will be pointed out. -->
@@ -11,7 +11,7 @@
     <!-- The base origin is offset from the world origin. -->
     <joint name="base_joint" type="fixed">
+        <origin xyz="1.5 1.0 0" rpy="0 0 0"/>
         <parent link="world"/>
         <child link="base_link"/>
-        <origin xyz="1.5 1.0 0.0" rpy="0.0 0.0 0.0"/>
     </joint>
     <!-- base_link is a large rectangular plate. Some things to note: -->
@@ -22,7 +22,7 @@
     <link name="base_link">
         <visual>
-            <origin xyz="0.0 0.0 0.05" rpy="0.0 0.0 0.0"/>
+            <origin xyz="0 0 0.05" rpy="0 0 0"/>
             <geometry>
-                <box size="2.5 1.5 0.1"/>
+                <box size="2.5 1.5 0.1" />
             </geometry>
             <material name="green">
@@ -31,13 +31,13 @@
         </visual>
         <collision>
-            <origin xyz="0.0 0.0 0.05" rpy="0.0 0.0 0.0"/>
+            <origin xyz="0 0 0.05" rpy="0 0 0"/>
             <geometry>
-                <box size="2.5 1.5 0.1"/>
+                <box size="2.5 1.5 0.1" />
             </geometry>
         </collision>
         <inertial>
-            <origin xyz="0.0 0.0 0.5" rpy="0.0 0.0 0.0"/>
-            <mass value="12"/>
-            <inertia ixx="2.26" ixy="0.0" ixz="0.0" iyy="6.26" iyz="0.0" izz="8.5"/>
+            <origin xyz="0 0 0.05" rpy="0 0 0"/>
+            <mass value="12" />
+            <inertia ixx="2.26" ixy="0.0" ixz="0.0" iyy="6.26" iyz="0.0" izz="8.5" />
         </inertial>
     </link>
@@ -47,9 +47,10 @@
     <!-- - We need to specify limits for the motion -->
     <joint name="slider_joint" type="prismatic">
+        <origin xyz="-1.25 0 0.1" rpy="0 0 0"/>
         <parent link="base_link"/>
         <child link="slider_link"/>
         <axis xyz="1 0 0"/>
         <limit lower="0" upper="2" velocity="100" effort="100"/>
-        <origin xyz="-1.25 0 0.1" rpy="0 0 0"/>
+        <dynamics damping="10.0" friction="10.0"/>
     </joint>
     <!-- slider_link is the box skimming across the top of the base. Its parameters are similar to the base_link, however: -->
@@ -58,18 +59,18 @@
     <link name="slider_link">
         <visual>
-            <origin xyz="0.0 0.0 0.075" rpy="0.0 0.0 0.0"/>
+            <origin xyz="0 0 0.075" rpy="0 0 0"/>
             <geometry>
-                <box size="0.5  0.25 0.15" />
+                <box size="0.5 0.25 0.15" />
             </geometry>
-            <material name="blue"/>
+            <material name="blue" />
         </visual>
         <collision>
-            <origin xyz="0.0 0.0 0.075" rpy="0.0 0.0 0.0"/>
+            <origin xyz="0 0 0.075" rpy="0 0 0"/>
             <geometry>
                 <box size="0.5 0.25 0.15" />
             </geometry>
         </collision>
-        <xacro:inertial_box mass="0.5" x="0.5" y="0.25" z="0.15" />
-            <origin xyz="0.0 0.0 0.075" rpy="0.0 0.0 0.0"/>
+        <xacro:inertial_box mass="0.5" x="0.5" y="0.25" z="0.15">
+            <origin xyz="0 0 0.075" rpy="0 0 0"/>
         </xacro:inertial_box>
     </link>
@@ -78,9 +79,10 @@
     <!-- - The upper limit uses xacro's mathematical features -->
     <joint name="arm_joint" type="revolute">
-        <origin xyz="0.25 0.0 0.15" rpy="0.0 0.0 0.0"/>
+        <origin xyz="0.25 0 0.15" rpy="0 0 0"/>
         <parent link="slider_link"/>
         <child link="arm_link"/>
         <axis xyz="0 -1 0"/>
-        <limit lower="0.0" upper="${pi/2}" effort="100" velocity="100"/>
+        <limit lower="0" upper="${pi/2}" velocity="100" effort="100"/>
+        <dynamics damping="10.0" friction="10.0"/>
     </joint>
     <!-- arm_link describes the arm -->
@@ -88,25 +90,25 @@
     <!-- - The visual/collision origin is set to halfway along the length (similar to the box), but also with a rotation (again using the mathematical features). -->
     <!--   This is because the cylinder extends along the Z axis by default, but we want it to be along the X axis (when the joint is at 0) -->
-    <xacro:property name="arm_length" value="1"/>
-    <xacro:property name="arm_radius" value="0.1"/>
+    <xacro:property name="arm_length" value="1" />
+    <xacro:property name="arm_radius" value="0.1" />
     <link name="arm_link">
         <visual>
-            <origin xyz="${arm_radius/2}" rpy="0.0 ${pi/2} 0.0"/>
+            <origin xyz="${arm_length/2} 0 0" rpy="0 ${pi/2} 0"/>
             <geometry>
-                <cylinder radius="${arm_radius}" length="${arm_length}"/>
+                <cylinder length="${arm_length}" radius="${arm_radius}" />
             </geometry>
-            <material name="orange"/>
+            <material name="orange" />
         </visual>
         <collision>
-            <origin xyz="${arm_radius/2}" rpy="0.0 ${pi/2} 0.0"/>
+            <origin xyz="${arm_length/2} 0 0" rpy="0 ${pi/2} 0"/>
             <geometry>
-                <cylinder radius="${arm_radius}" length="${arm_length}"/>
+                <cylinder length="${arm_length}" radius="${arm_radius}" />
             </geometry>
         </collision>
         <xacro:inertial_cylinder mass="1.0" length="${arm_length}" radius="${arm_radius}">
-            <origin xyz="${arm_length/2} 0.0 0.0" rpy="0.0 ${pi/2} 0.0"/>
+            <origin xyz="${arm_length/2} 0 0" rpy="0 ${pi/2} 0"/>
         </xacro:inertial_cylinder>
     </link>
-     <!-- camera_joint describes where the camera is relative to the arm -->
+    <!-- camera_joint describes where the camera is relative to the arm -->
     <!-- - Even though the camera isn't moving relative to the arm, it will probably be helpful to have its own link/frame rather than just adding more visuals to the arm -->
     <!-- - For this example, the camera_link origin will be at the centre of the camera's "sensor" -->
